Commit message: Phase 2: Jezero delta terrain from HiRISE, waypoints on Perseverance's route
Adds world:=jezero_delta (Harmonic): 256 m of the Jezero delta front, 65.8 m
of relief, cropped from the USGS Mars 2020 HiRISE DTM mosaic (1 m/px) by
reading a ~22 MB window over HTTP. Waypoints are Perseverance's positions on
sols 437, 441, 448, 455, 461 from NASA's traverse data; their recorded
elevations match the DTM within 0.1-0.4 m. Mars gravity, 16-bit heightmap,
spawn pose and waypoints in worlds/jezero_delta.yaml for Phase 3.
terrain/build_jezero_delta.sh regenerates it all.

Model fixes: the sim passes wheel_radius 0.082 to the rover node (forward
speed 0.327 -> 0.300 m/s for 0.3 commanded), and wheel_mu:= (default 0.7)
applies friction through <gazebo reference>, which survives URDF->SDF where
upstream's <surface> block didn't.

Verified: settles at the DTM height of the spawn (3.24 vs 3.29 m), holds on
a 7 deg slope, and drives 33.6 m up to within 1.7 m of the sol 441 waypoint.
RTF 21-22x unthrottled on the terrain (gz /stats).

Tried and dropped: the rocker differential as a URDF mimic joint. DART in
Harmonic rejects mimic constraints and the body flopped to -35 deg; rockers
stay fixed as upstream. Findings in PLAN.md.

Launch: world:= takes a name or path; realtime:=/step:= now apply to any
world; empty worlds renamed. Tools: drive_test.py; bench.py reads RTF from
gz /stats and waits for DDS discovery before timing.

Co-Authored-By: Claude Opus 5.5 <noreply@anthropic.com>
Claude-Session: https://claude.ai/code/session_01XjDodjUyBxSte15sfszJGN

File: ros_ws/src/osr_gz/urdf/osr.urdf.xacro (robot description, xacro)
@@ -14,10 +14,18 @@
   - sim:=classic|harmonic selects the ros2_control / IMU plugins (osr_gz.xacro).
   - Upstream's <surface><friction> inside <collision> is dropped: URDF can't carry
-    it, and `gz sdf -p` confirms it never reached the simulator. Wheels run on the
-    simulator's default friction, as they always have.
+    it, and `gz sdf -p` confirms it never reached the simulator. wheel_mu:= sets
+    it properly through <gazebo reference> (isotropic: upstream's mu2 of 0.3 has
+    no defined direction without fdir1, so each engine would pick its own).
+  - The rocker pivots stay fixed, as upstream has them; only the bogies
+    articulate. The OSR's differential (left rocker = -right) can't be expressed
+    here: URDF <mimic> converts to SDF fine, but gz-physics DART in Harmonic
+    rejects mimic constraints ("the chosen physics engine does not support mimic
+    constraints"), leaving the body free to pitch (it flopped to -35 deg). See
+    PLAN.md, Phase 2 results.
 -->
 <robot xmlns:xacro="http://www.ros.org/wiki/xacro" name="rover">
     <xacro:arg name="sim" default="classic"/>
     <xacro:arg name="collision" default="primitive"/>
+    <xacro:arg name="wheel_mu" default="0.7"/>
     <xacro:property name="primitive" value="${'$(arg collision)' == 'primitive'}"/>
     <xacro:property name="mesh_dir" value="file://$(find osr_gz)/meshes"/>
@@ -137,11 +145,9 @@
             <primitive_collision/>
         </xacro:mesh_link>
-        <!-- Upstream has the rocker pivot fixed; only the bogie articulates.
-             Kept as-is for parity with Phase 0. -->
+        <!-- Fixed, as upstream: see the header comment. -->
         <joint name="rocker_bogie_joint_${prefix}_1" type="fixed">
             <parent link="body_axis_link_${prefix}"/>
             <origin rpy="0 0 0" xyz="0.016004 ${dir*0.071485} 0.001353"/>
             <child link="rocker_bogie_link_${prefix}_1"/>
-            <limit effort="10000.0" velocity="0.5" lower="-0.5" upper="0.5"/>
             <axis xyz="0 1 0"/>
         </joint>
@@ -203,4 +209,8 @@
     <!-- The six driven wheels. -->
     <xacro:macro name="wheel_tyre" params="name dir origin">
+        <gazebo reference="${name}">
+            <mu1>$(arg wheel_mu)</mu1>
+            <mu2>$(arg wheel_mu)</mu2>
+        </gazebo>
         <!-- Right side is yawed 180 degrees; dir mirrors the offset so the tyre
              centre stays inboard on both sides. -->

Commit message: Phase 4 (in progress): PPO tooling, boulder fields, route goals
Training: CPU-only torch + Stable-Baselines3 + TensorBoard in the image;
train/train.py (PPO over SubprocVecEnv, VecNormalize saved with each
checkpoint, outcome-rate logging, --resume); eval/evaluate.py (policy vs
baseline on identical held-out spawns: plain / hard / unseen segment);
tools/tb_summary.py.

Finding: on the plain delta the baseline is ~optimal (100%, 0.30 m/s), and
ppo_v1 (1.0M steps) is slower and memorised its segments (42% on the unseen
one). The crater rim (jezero_rim, added) is steep but not hard in this sim.

Boulder fields: terrain/add_rocks.py sizes rocks with the Golombek-Rapp Mars
rock-abundance model (coverage matches it: 2.0% vs 1.9% at k=0.05) and bakes
them into a 2049px heightmap. As models, 2,544 rocks ran at 0.4x real time;
baked, 12.8x. Rocks block, deflect and flip the rover by size, and the
baseline drops to 42% on the hard variant. Rocker/bogie/bracket beams get
box collisions (flat-ground behaviour unchanged).

Env: spawn_jitter, rock_patch (0.4 m terrain patch that sees rocks),
goal_mode='route' (random start/goal pairs along the route), spawns and
goals kept off rocks.

ppo_rocks (k=0.05, route goals, rock patch) is training; results to follow.

Co-Authored-By: Claude Opus 5.5 <noreply@anthropic.com>
Claude-Session: https://claude.ai/code/session_01XjDodjUyBxSte15sfszJGN

File: ros_ws/src/osr_gz/urdf/osr.urdf.xacro (robot description, xacro)
@@ -8,8 +8,8 @@
   - collision:=mesh       upstream behaviour: every link collides with its full STL
                           (~1.4M triangles total; RTF 0.25 in jezero-lab Phase 0).
-    collision:=primitive  wheels are cylinders, the body is a box. Structural links
-                          that can't reach flat ground (arms, turnbuckles, rockers,
-                          steering brackets) get no collision. Revisit for rough
-                          terrain in Phase 2.
+    collision:=primitive  wheels are cylinders, the body is a box, and the rocker,
+                          bogie, and steering-bracket beams are 4 cm boxes between
+                          their joints (so the rover can high-centre on rocks).
+                          Arms and turnbuckles, inside the body's footprint, get none.
   - sim:=classic|harmonic selects the ros2_control / IMU plugins (osr_gz.xacro).
   - Upstream's <surface><friction> inside <collision> is dropped: URDF can't carry
@@ -40,4 +40,16 @@
     <xacro:include filename="$(find osr_gz)/urdf/osr_gz.xacro"/>
     <xacro:osr_gz_plugins sim="$(arg sim)"/>
+    <!-- A structural beam as a box from p1 to p2 (link frame, x-z plane; the
+         y offsets involved are millimetres). Used for primitive collisions on
+         the rockers, bogies, and steering brackets, so the rover can high-centre
+         on rocks. Endpoints are the joint origins the links connect. -->
+    <xacro:property name="beam_w" value="0.04"/>
+    <xacro:macro name="beam" params="x1 z1 x2 z2">
+        <collision>
+            <origin xyz="${(x1 + x2) / 2} 0 ${(z1 + z2) / 2}"
+                    rpy="0 ${atan2(-(z2 - z1), x2 - x1)} 0"/>
+            <geometry><box size="${sqrt((x2 - x1)**2 + (z2 - z1)**2)} ${beam_w} ${beam_w}"/></geometry>
+        </collision>
+    </xacro:macro>
     <!-- Visual always uses the mesh. Collision uses the mesh only in mesh mode;
          the caller supplies a primitive via the block, or nothing. -->
@@ -143,5 +155,8 @@
                          mass="7" ixx="0.24701126860819052" iyy="3.544526366681435" izz="3.335915098740816">
             <origin rpy="0 0 0" xyz="0 0 0.0"/>
-            <primitive_collision/>
+            <primitive_collision>
+                <xacro:beam x1="0" z1="0" x2="0.099618" z2="-0.091275"/>
+                <xacro:beam x1="0" z1="0" x2="-0.311763" z2="-0.030379"/>
+            </primitive_collision>
         </xacro:mesh_link>
         <!-- Fixed, as upstream: see the header comment. -->
@@ -155,5 +170,8 @@
                          mass="3" ixx="0.51733003028693055" iyy="1.1690895987181758" izz="0.6934262363396754">
             <origin rpy="0 0 0" xyz="0 0 0.0"/>
-            <primitive_collision/>
+            <primitive_collision>
+                <xacro:beam x1="0" z1="0" x2="0.170113" z2="0.076721"/>
+                <xacro:beam x1="0" z1="0" x2="-0.101456" z2="-0.100276"/>
+            </primitive_collision>
         </xacro:mesh_link>
         <joint name="rocker_bogie_joint_${prefix}_2" type="revolute">
@@ -172,5 +190,7 @@
                          mass="0.8" ixx="0.002865290876023045" iyy="0.004329299643338258" izz="0.0018192303726865125">
             <origin rpy="0 0 ${dir*-1.57}" xyz="0 0 0.0"/>
-            <primitive_collision/>
+            <primitive_collision>
+                <xacro:beam x1="0" z1="0" x2="0.006231" z2="${-0.169991 + wheel_r}"/>
+            </primitive_collision>
         </xacro:mesh_link>
         <joint name="front_wheel_joint_${prefix}" type="revolute">
@@ -195,5 +215,7 @@
                          mass="0.8" ixx="0.002865290876023045" iyy="0.004329299643338258" izz="0.0018192303726865125">
             <origin rpy="0 0 ${-dir*1.57}" xyz="0 0 0.0"/>
-            <primitive_collision/>
+            <primitive_collision>
+                <xacro:beam x1="0" z1="0" x2="-0.000203" z2="${-0.160678 + wheel_r}"/>
+            </primitive_collision>
         </xacro:mesh_link>
         <joint name="rear_wheel_joint_${prefix}" type="revolute">

Commit message: Phase 5: path plots, chase-camera video, ROCm measured and skipped
ROCm: tools/profile_train.py shows the PPO network update is 2% of training
wall time (0.18 s of a 9.6 s iteration); the rest is the simulators in
lockstep. A GPU could make training at most 1.02x faster, so it isn't used.
The real levers (coarser step, more simulators, no reset stalls) are noted.

eval/plot_paths.py draws baseline and policy paths per held-out spawn over
the boulder terrain. They show how ppo_rocks fails on the unseen segment:
it veers north-east off the goal bearing and stalls at a scarp the baseline
drives straight across.

eval/record.py adds an optional chase camera (Sensors system, ogre2 on the
RX 7600) and streams frames to ffmpeg; eval/make_demo.sh makes side-by-side
baseline/policy videos with outcome captions. Recordings reproduce the
evaluation exactly. Rendering needed the OSRF ogre2 plugin plus aliases and
GZ_RENDERING_RESOURCE_PATH pointed at ROS's vendor shaders (same 8.2.3).

Docs: PLAN.md Phase 5 results and where the project stands; README shows
the result, usage, and plots from docs/media/.

Co-Authored-By: Claude Opus 5.5 <noreply@anthropic.com>
Claude-Session: https://claude.ai/code/session_01XjDodjUyBxSte15sfszJGN

File: ros_ws/src/osr_gz/urdf/osr.urdf.xacro (robot description, xacro)
@@ -28,4 +28,5 @@
     <xacro:arg name="collision" default="primitive"/>
     <xacro:arg name="wheel_mu" default="0.7"/>
+    <xacro:arg name="camera" default="false"/>
     <xacro:property name="primitive" value="${'$(arg collision)' == 'primitive'}"/>
     <xacro:property name="mesh_dir" value="file://$(find osr_gz)/meshes"/>
@@ -40,4 +41,7 @@
     <xacro:include filename="$(find osr_gz)/urdf/osr_gz.xacro"/>
     <xacro:osr_gz_plugins sim="$(arg sim)"/>
+    <xacro:if value="$(arg camera)">
+        <xacro:chase_camera/>
+    </xacro:if>
     <!-- A structural beam as a box from p1 to p2 (link frame, x-z plane; the
          y offsets involved are millimetres). Used for primitive collisions on

File: ros_ws/src/osr_gz/urdf/osr_gz.xacro (robot description, xacro)
@@ -29,4 +29,22 @@
       <state_interface name="effort"/>
     </joint>
+  </xacro:macro>
+  <!-- Chase camera for recordings (sim:=gym camera:=true): behind and above the
+       body, tilted down, following the rover. Needs the world's Sensors system,
+       which jezero_env adds when recording. -->
+  <xacro:macro name="chase_camera">
+    <gazebo reference="base_link">
+      <sensor name="chase_cam" type="camera">
+        <pose>-1.6 0 0.9 0 0.38 0</pose>
+        <always_on>true</always_on>
+        <update_rate>15</update_rate>
+        <topic>chase_cam</topic>
+        <camera>
+          <horizontal_fov>1.2</horizontal_fov>
+          <image><width>960</width><height>540</height><format>R8G8B8</format></image>
+          <clip><near>0.1</near><far>300</far></clip>
+        </camera>
+      </sensor>
+    </gazebo>
   </xacro:macro>
   <xacro:macro name="osr_gz_plugins" params="sim">

Commit message: upstream: bump osr-rover-code to b874497 (PR #230 merged, PR #232 rotate-in-place fix)
PR #230 (ours) changes only upstream's Classic osr_gazebo; osr_gz already applied
friction this way. PR #232 fixes swapped d2/d3 corner angles in rotate-in-place,
which jezero_env/sim.py calls. Benched old vs new image: rotate rate within
scatter, driving episode bit-identical, so no experiment needs re-running.

Co-Authored-By: Claude Opus 5.5 <noreply@anthropic.com>
Claude-Session: https://claude.ai/code/session_0172PGD2SRgtSEybhnxsVT4z

File: ros_ws/src/osr_gz/urdf/osr.urdf.xacro (robot description, xacro)
@@ -13,8 +13,8 @@
                           Arms and turnbuckles, inside the body's footprint, get none.
   - sim:=classic|harmonic selects the ros2_control / IMU plugins (osr_gz.xacro).
-  - Upstream's <surface><friction> inside <collision> is dropped: URDF can't carry
-    it, and `gz sdf -p` confirms it never reached the simulator. wheel_mu:= sets
-    it properly through <gazebo reference> (isotropic: upstream's mu2 of 0.3 has
-    no defined direction without fdir1, so each engine would pick its own).
+  - Friction: wheel_mu:= sets it through <gazebo reference> (isotropic). Before
+    upstream b874497 (PR #230), upstream put it in <surface><friction> inside
+    <collision>, which URDF can't carry, so it never reached the simulator
+    (`gz sdf -p`); its mu2 of 0.3 also had no defined direction without fdir1.
   - The rocker pivots stay fixed, as upstream has them; only the bogies
     articulate. The OSR's differential (left rocker = -right) can't be expressed
